Commit message: Roslaunch Gazebo + add body inertia

File: sim_tutorial/description/urdf/cybertruck.urdf.xacro (robot description, xacro)
@@ -1,4 +1,7 @@
 <?xml version="1.0"?>
 <robot name="cybertruck" xmlns:xacro="http://ros.org/wiki/xacro">
+     <!-- Includes -->
+    <xacro:include filename="$(find description)/urdf/constants.xacro"/>
+    <xacro:include filename="$(find description)/urdf/inertias.xacro"/>
     <link name="base_link"/>
     <!-- body_link -->
@@ -16,4 +19,7 @@
             </geometry>
         </collision>
+        <inertial>
+            <xacro:body_inertial m="${body_mass}" l="${body_length}" w="${body_width}" h="${body_height}"/>
+        </inertial>
     </link>
     <!-- Body joint -->
