Commit message: Added wheels in Gazebo

File: sim_tutorial/description/urdf/inertias.xacro (robot description, xacro)
@@ -13,4 +13,12 @@
     <!-- Wheel -->
     <!-- NOTE: wheels are radially symmetric around the x-axis -->
-    <!-- TODO: define a macro for the inertial of a wheel (can approx as a cylinder) -->
+    <!-- TODO: define a macro for the inertial of a wheel (can approx as a cylinder)  HEIGHT ALONG THE X AXIS -->
+    <xacro:macro name="wheel_inertial" params="m r h">
+        <mass value="${m}"/>
+        <inertia
+            ixx="${m*r*r/2}" ixy="0" ixz="0"
+            iyy="${m*(3*r*r + h*h)/12}" iyz="0"
+            izz="${m*(3*r*r + h*h)/12}"
+        />
+    </xacro:macro>
 </robot>

File: sim_tutorial/description/urdf/wheels.urdf.xacro (robot description, xacro)
@@ -19,4 +19,8 @@
                 </geometry>
             </collision>
+            <!-- Inertials -->
+            <inertial>
+                <xacro:wheel_inertial m="${wheel_mass}" r="${wheel_radius}" h="${wheel_width}"/>
+            </inertial>
         </link>
         <!-- Wheel joint -->
